File: content/electronics/components/power-regulators/charge-pumps/charge-pump-voltage-doubler-simulation/charge-pump-voltage-doubler-simulation.sch (KiCad schematic (older format))
At the start: 7 parts

Commit message: Added more simulation data to the charge pumps page.
Parts:
- removed D2: 1N4148, symbol charge-pump-voltage-doubler-simulation-rescue:D-rectifier_schlib-charge-pump-vo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
- added D2: 1N5817, symbol charge-pump-voltage-doubler-simulation-rescue:D-rectifier_schlib-charge-pump-vo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
- C1, C2: symbol charge-pump-voltage-doubler-simulation-rescue:C-rectifier_schlib-charge-pump-voltage-doubler-simulation-rescue -> charge-pump-voltage-doubler-simulation-rescue:C-rectifier_schlib-charge-pump-voltage-doubler-simulation-rescue-charge-p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
- D1: value 1N4148 -> 1N5817; symbol charge-pump-voltage-doubler-simulation-rescue:D-rectifier_schlib-charge-pump-voltage-doubler-simulation-rescue -> charge-pump-voltage-doubler-simulation-rescue:D-rectifier_schlib-charge-pump-voltage-doubler-simulation-rescue-charge-p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; Spice_Lib_File (none) -> 1n5817.lib; Spice_Model (none) -> 1N5817; Spice_Netlist_Enabled (none) -> Y; Spice_Primitive D -> X
- R2: value 100k -> 100R; symbol charge-pump-voltage-doubler-simulation-rescue:R-rectifier_schlib-charge-pump-voltage-doubler-simulation-rescue -> charge-pump-voltage-doubler-simulation-rescue:R-rectifier_schlib-charge-pump-voltage-doubler-simulation-rescue-charge-p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
- V1, V2: symbol charge-pump-voltage-doubler-simulation-rescue:VSOURCE-rectifier_schlib-charge-pump-voltage-doubler-simulation-rescue -> charge-pump-voltage-doubler-simulation-rescue:VSOURCE-rectifier_schlib-charge-pump-voltage-doubler-simulation-rescue-ch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
Changed lines of the file:
@@
 $EndDescr
 $Comp
-L charge-pump-voltage-doubler-simulation-rescue:VSOURCE-rectifier_schlib-charge-pump-voltage-doubler-simulation-rescue V2
+L charge-pump-voltage-doubler-simulation-rescue:VSOURCE-rectifier_schlib-charge-pump-voltage-doubler-simulation-rescue-charge-pump-voltage-doubler-simulation-rescue-charge-pump-voltage-doubler-simulation-rescue V2
 U 1 1 57336052
 P 4200 4550
@@
 $EndComp
 $Comp
-L charge-pump-voltage-doubler-simulation-rescue:GND-rectifier_schlib-charge-pump-voltage-doubler-simulation-rescue #PWR01
+L charge-pump-voltage-doubler-simulation-rescue:GND-rectifier_schlib-charge-pump-voltage-doubler-simulation-rescue-charge-pump-voltage-doubler-simulation-rescue-charge-pump-voltage-doubler-simulation-rescue #PWR01
 U 1 1 573360D3
 P 4200 4850
@@
 $EndComp
 $Comp
-L charge-pump-voltage-doubler-simulation-rescue:D-rectifier_schlib-charge-pump-voltage-doubler-simulation-rescue D1
+L charge-pump-voltage-doubler-simulation-rescue:D-rectifier_schlib-charge-pump-voltage-doubler-simulation-rescue-charge-pump-voltage-doubler-simulation-rescue-charge-pump-voltage-doubler-simulation-rescue D1
 U 1 1 573361B8
 P 4500 3650
 F 0 "D1" H 4500 3435 50  0000 C CNN
-F 1 "1N4148" H 4500 3526 50  0000 C CNN
+F 1 "1N5817" H 4500 3526 50  0000 C CNN
 F 2 "" H 4500 3650 50  0000 C CNN
 F 3 "" H 4500 3650 50  0000 C CNN
 F 4 "Value" H 4500 3650 60  0001 C CNN "Fieldname"
-F 5 "D" H 4500 3650 60  0001 C CNN "Spice_Primitive"
+F 5 "X" H 4500 3650 60  0001 C CNN "Spice_Primitive"
 F 6 "2 1" H 4500 3650 60  0001 C CNN "Spice_Node_Sequence"
+F 7 "1n5817.lib" H 4500 3650 50  0001 C CNN "Spice_Lib_File"
+F 8 "1N5817" H 4500 3650 50  0001 C CNN "Spice_Model"
+F 9 "Y" H 4500 3650 50  0001 C CNN "Spice_Netlist_Enabled"
 	1    4500 3650
 	-1   0    0    1
 $EndComp
 $Comp
-L charge-pump-voltage-doubler-simulation-rescue:C-rectifier_schlib-charge-pump-voltage-doubler-simulation-rescue C1
+L charge-pump-voltage-doubler-simulation-rescue:C-rectifier_schlib-charge-pump-voltage-doubler-simulation-rescue-charge-pump-voltage-doubler-simulation-rescue-charge-pump-voltage-doubler-simulation-rescue C1
 U 1 1 5733628F
 P 5350 4000
@@
 $EndComp
 $Comp
-L charge-pump-voltage-doubler-simulation-rescue:R-rectifier_schlib-charge-pump-voltage-doubler-simulation-rescue R2
+L charge-pump-voltage-doubler-simulation-rescue:R-rectifier_schlib-charge-pump-voltage-doubler-simulation-rescue-charge-pump-voltage-doubler-simulation-rescue-charge-pump-voltage-doubler-simulation-rescue R2
 U 1 1 573362F7
 P 5700 4000
 F 0 "R2" H 5630 3954 50  0000 R CNN
-F 1 "100k" H 5630 4045 50  0000 R CNN
+F 1 "100R" H 5630 4045 50  0000 R CNN
 F 2 "" V 5630 4000 50  0000 C CNN
 F 3 "" H 5700 4000 50  0000 C CNN
@@
 	5350 3650 5700 3650
 $Comp
-L charge-pump-voltage-doubler-simulation-rescue:VSOURCE-rectifier_schlib-charge-pump-voltage-doubler-simulation-rescue V1
+L charge-pump-voltage-doubler-simulation-rescue:VSOURCE-rectifier_schlib-charge-pump-voltage-doubler-simulation-rescue-charge-pump-voltage-doubler-simulation-rescue-charge-pump-voltage-doubler-simulation-rescue V1
 U 1 1 5FD5E984
 P 3950 3850
@@
 $EndComp
 $Comp
-L charge-pump-voltage-doubler-simulation-rescue:C-rectifier_schlib-charge-pump-voltage-doubler-simulation-rescue C2
+L charge-pump-voltage-doubler-simulation-rescue:C-rectifier_schlib-charge-pump-voltage-doubler-simulation-rescue-charge-pump-voltage-doubler-simulation-rescue-charge-pump-voltage-doubler-simulation-rescue C2
 U 1 1 5FD681FD
 P 4800 4000
@@
 	1    0    0    -1
 $EndComp
-$Comp
-L charge-pump-voltage-doubler-simulation-rescue:D-rectifier_schlib-charge-pump-voltage-doubler-simulation-rescue D2
-U 1 1 5FD68D10
-P 5050 3650
-F 0 "D2" H 5050 3435 50  0000 C CNN
-F 1 "1N4148" H 5050 3526 50  0000 C CNN
-F 2 "" H 5050 3650 50  0000 C CNN
-F 3 "" H 5050 3650 50  0000 C CNN
-F 4 "Value" H 5050 3650 60  0001 C CNN "Fieldname"
-F 5 "D" H 5050 3650 60  0001 C CNN "Spice_Primitive"
-F 6 "2 1" H 5050 3650 60  0001 C CNN "Spice_Node_Sequence"
-	1    5050 3650
-	-1   0    0    1
-$EndComp
-Wire Wire Line
-	4650 3650 4800 3650
 Wire Wire Line
 	4800 3850 4800 3650
@@
 	4200 4750 4200 4850
 $Comp
-L charge-pump-voltage-doubler-simulation-rescue:GND-rectifier_schlib-charge-pump-voltage-doubler-simulation-rescue #PWR?
+L charge-pump-voltage-doubler-simulation-rescue:GND-rectifier_schlib-charge-pump-voltage-doubler-simulation-rescue-charge-pump-voltage-doubler-simulation-rescue-charge-pump-voltage-doubler-simulation-rescue #PWR?
 U 1 1 5FD69C41
 P 3950 4050
@@
 $EndComp
 $Comp
-L charge-pump-voltage-doubler-simulation-rescue:GND-rectifier_schlib-charge-pump-voltage-doubler-simulation-rescue #PWR?
+L charge-pump-voltage-doubler-simulation-rescue:GND-rectifier_schlib-charge-pump-voltage-doubler-simulation-rescue-charge-pump-voltage-doubler-simulation-rescue-charge-pump-voltage-doubler-simulation-rescue #PWR?
 U 1 1 5FD6A33F
 P 5500 4350
@@
 vin
 Wire Wire Line
+	4650 3650 4800 3650
+Wire Wire Line
 	3950 3650 4350 3650
+$Comp
+L charge-pump-voltage-doubler-simulation-rescue:D-rectifier_schlib-charge-pump-voltage-doubler-simulation-rescue-charge-pump-voltage-doubler-simulation-rescue-charge-pump-voltage-doubler-simulation-rescue D2
+U 1 1 5FDBF038
+P 5050 3650
+F 0 "D2" H 5050 3435 50  0000 C CNN
+F 1 "1N5817" H 5050 3526 50  0000 C CNN
+F 2 "" H 5050 3650 50  0000 C CNN
+F 3 "" H 5050 3650 50  0000 C CNN
+F 4 "Value" H 5050 3650 60  0001 C CNN "Fieldname"
+F 5 "X" H 5050 3650 60  0001 C CNN "Spice_Primitive"
+F 6 "2 1" H 5050 3650 60  0001 C CNN "Spice_Node_Sequence"
+F 7 "1n5817.lib" H 5050 3650 50  0001 C CNN "Spice_Lib_File"
+F 8 "1N5817" H 5050 3650 50  0001 C CNN "Spice_Model"
+F 9 "Y" H 5050 3650 50  0001 C CNN "Spice_Netlist_Enabled"
+	1    5050 3650
+	-1   0    0    1
+$EndComp
 $EndSCHEMATC
