File: content/electronics/circuit-design/analogue-filters/low-pass-sallen-key-bessel/schematic-simulation.sch (KiCad schematic (older format))
At the start: 8 parts, among them U1 AD8051

Commit message: Added a Bessel optimized low-pass Sallen-Key filter simulation schematic and added the results of the comparison plots.
Parts:
- C1: value 88n -> 15n
- R1: value 4.99k -> 7.15k
- R2: value 12.1k -> 14.3k
Changed lines of the file:
@@
 P 4050 3650
 F 0 "R1" V 3845 3650 50  0000 C CNN
-F 1 "4.99k" V 3936 3650 50  0000 C CNN
+F 1 "7.15k" V 3936 3650 50  0000 C CNN
 F 2 "" H 4150 2950 50  0001 L CNN
 F 3 "" H 4050 3650 50  0001 L CNN
@@
 P 4800 3150
 F 0 "C1" V 4548 3150 50  0000 C CNN
-F 1 "88n" V 4639 3150 50  0000 C CNN
+F 1 "15n" V 4639 3150 50  0000 C CNN
 F 2 "" H 5000 2350 50  0001 L CNN
 F 3 "" H 4800 3150 50  0001 L CNN
@@
 P 4500 3650
 F 0 "R2" V 4295 3650 50  0000 C CNN
-F 1 "12.1k" V 4386 3650 50  0000 C CNN
+F 1 "14.3k" V 4386 3650 50  0000 C CNN
 F 2 "" H 4600 2950 50  0001 L CNN
 F 3 "" H 4500 3650 50  0001 L CNN
