File: content/electronics/components/oscillators/ring-oscillator-single/simulation.sch (KiCad schematic (older format))
At the start: 2 parts, among them U1 74HCU04

Commit message: Working on the single NOT gate ring oscillator simulation circuit.
Parts:
- added R1: 10k, symbol mbedded-ninja-kicad-symbols-sim:10k
Connections:
- net GND: now also R1.2
- net VOUT renamed OUT
- net OUT: now also R1.1
Changed lines of the file:
@@
 Wire Wire Line
 	3300 2400 3350 2400
-Text Label 3350 2400 0    50   ~ 0
-VOUT
+Text GLabel 3350 2400 2    50   Input ~ 0
+OUT
+$Comp
+L mbedded-ninja-kicad-symbols-sim:10k R1
+U 1 1 6095F44B
+P 3300 2550
+F 0 "R1" H 3368 2596 50  0000 L CNN
+F 1 "10k" H 3368 2505 50  0000 L CNN
+F 2 "" H 3400 1850 50  0001 L CNN
+F 3 "" H 3300 2550 50  0001 L CNN
+F 4 "R" H 3450 2400 50  0001 C CNN "Spice_Primitive"
+	1    3300 2550
+	1    0    0    -1
+$EndComp
+Connection ~ 3300 2400
+$Comp
+L power:GND #PWR?
+U 1 1 60960813
+P 3300 2700
+F 0 "#PWR?" H 3300 2450 50  0001 C CNN
+F 1 "GND" H 3305 2527 50  0000 C CNN
+F 2 "" H 3300 2700 50  0001 C CNN
+F 3 "" H 3300 2700 50  0001 C CNN
+	1    3300 2700
+	1    0    0    -1
+$EndComp
 $EndSCHEMATC

Commit message: Added schematics and simulation results for a three stage ring oscillator.
Connections:
- net GND: no longer U1.1
- net OUT: now also U1.1
Other:
- note added: ".tran 100f 10n"
- note removed: ".tran 0.1 1"
- moved on the sheet: R1
Changed lines of the file:
@@
 Text GLabel 4150 1850 0    50   Input ~ 0
 +5V
-$Comp
-L power:GND #PWR0103
-U 1 1 6094EE4D
-P 2700 2400
-F 0 "#PWR0103" H 2700 2150 50  0001 C CNN
-F 1 "GND" H 2705 2227 50  0000 C CNN
-F 2 "" H 2700 2400 50  0001 C CNN
-F 3 "" H 2700 2400 50  0001 C CNN
-	1    2700 2400
-	1    0    0    -1
-$EndComp
 Text Notes 2400 2900 0    50   ~ 0
-.tran 0.1 1
+.tran 100f 10n
 $Comp
 L mbedded-ninja-kicad-symbols-sim:74HCU04 U1
@@
 L mbedded-ninja-kicad-symbols-sim:10k R1
 U 1 1 6095F44B
-P 3300 2550
-F 0 "R1" H 3368 2596 50  0000 L CNN
-F 1 "10k" H 3368 2505 50  0000 L CNN
-F 2 "" H 3400 1850 50  0001 L CNN
-F 3 "" H 3300 2550 50  0001 L CNN
-F 4 "R" H 3450 2400 50  0001 C CNN "Spice_Primitive"
-	1    3300 2550
+P 3300 2800
+F 0 "R1" H 3368 2846 50  0000 L CNN
+F 1 "10k" H 3368 2755 50  0000 L CNN
+F 2 "" H 3400 2100 50  0001 L CNN
+F 3 "" H 3300 2800 50  0001 L CNN
+F 4 "R" H 3450 2650 50  0001 C CNN "Spice_Primitive"
+	1    3300 2800
 	1    0    0    -1
 $EndComp
-Connection ~ 3300 2400
 $Comp
 L power:GND #PWR?
 U 1 1 60960813
-P 3300 2700
-F 0 "#PWR?" H 3300 2450 50  0001 C CNN
-F 1 "GND" H 3305 2527 50  0000 C CNN
-F 2 "" H 3300 2700 50  0001 C CNN
-F 3 "" H 3300 2700 50  0001 C CNN
-	1    3300 2700
+P 3300 2950
+F 0 "#PWR?" H 3300 2700 50  0001 C CNN
+F 1 "GND" H 3305 2777 50  0000 C CNN
+F 2 "" H 3300 2950 50  0001 C CNN
+F 3 "" H 3300 2950 50  0001 C CNN
+	1    3300 2950
 	1    0    0    -1
 $EndComp
+Wire Wire Line
+	2700 2400 2700 2650
+Wire Wire Line
+	2700 2650 3300 2650
+Wire Wire Line
+	3300 2650 3300 2400
+Connection ~ 3300 2400
+Connection ~ 3300 2650
 $EndSCHEMATC
